File: dronePCB/dronePCB.kicad_pcb (KiCad board)
At the start: 6 copper layers, 196 parts, among them IC1 STUSB4500QTR, IC2 MP2338GTL-Z, IC3 DPS368XTSA1, IC4 ICM-42688-P, J1 BM03B-SRSS-TB, J10 DVR, J11 Strobe top, J12 Strobe bottom, J13 ToF400C, J14 ToF400C, J15 ToF400C, J16 ToF400C, J17 ToF400C, J18 DSHOT, J19 ESC_POW, J2 USB_C_Receptacle, J3 103AT-2 10k, J4 XT30, J5 JST, J6 Camera, J7 VID_ANT, J8 GEP-M10Q, J9 Avatar GMx, Q1 BSS138, Q2 BSS138, SW1 SW_BOOT, SW2 SW_RESET, SW3 SW_CHG_RST, U1 RP2350_80QFN, U10 TF-01A, U2 W25Q128JVPIQ, U3 APS6404L-3SQR-ZR, U4 BQ25792RQMR, U5 NCP1117-3.3_SOT223, U6 BQ76920PW, U7 E28-2G4M12SX, U8 AT7456E, U9 TX5823, X1 OT2EL4C4JI-111OLP-27M, Y1 ABM8-272-T3

Commit message: Finished PCB
Parts:
- added SW4: CJS-1200TB1, droneParts:CJS1200TB1, B.Cu at (153.0, 140.3)
- added SW5: CJS-1200TB1, droneParts:CJS1200TB1, B.Cu at (156.7, 133.1)
- added SW6: CJS-1200TB1, droneParts:CJS1200TB1, B.Cu at (160.6, 140.4)
- C70, C72, C73, C79, C80, C82, C83, C84, C85, C86, C87, C88, C89, C90, J6, R11, R12, R47, R48, R49, U10: moved to B.Cu
- C78: footprint Capacitor_SMD:C_0805_2012Metric_Pad1.18x1.45mm_HandSolder -> Capacitor_SMD:C_Elec_3x5.4
- D4: footprint LED_SMD:LED_0201_0603Metric_Pad0.64x0.40mm_HandSolder -> LED_SMD:LED_0805_2012Metric_Pad1.15x1.40mm_HandSolder
- J1: footprint Connector_JST:JST_PH_B2B-PH-SM4-TB_1x02-1MP_P2.00mm_Vertical -> Connector_JST:JST_SH_BM03B-SRSS-TB_1x03-1MP_P1.00mm_Vertical
- J10: footprint Connector_JST:JST_PH_S3B-PH-SM4-TB_1x03-1MP_P2.00mm_Horizontal -> Connector_JST:JST_PH_B3B-PH-SM4-TB_1x03-1MP_P2.00mm_Vertical; moved to B.Cu
- J11, J12: footprint Connector_JST:JST_PH_S2B-PH-SM4-TB_1x02-1MP_P2.00mm_Horizontal -> Connector_JST:JST_PH_B2B-PH-SM4-TB_1x02-1MP_P2.00mm_Vertical
- J13, J14, J15, J16, J17: footprint Connector_JST:JST_PH_S6B-PH-SM4-TB_1x06-1MP_P2.00mm_Horizontal -> Connector_JST:JST_PH_B6B-PH-SM4-TB_1x06-1MP_P2.00mm_Vertical; moved to B.Cu
- J18, J9: footprint Connector_JST:JST_PH_S8B-PH-SM4-TB_1x08-1MP_P2.00mm_Horizontal -> Connector_JST:JST_PH_B8B-PH-SM4-TB_1x08-1MP_P2.00mm_Vertical; moved to B.Cu
- moved D4 123.3 mm to (149.2, 54.3)
- moved H1 89.0 mm to (122.3, 54.3)
- moved J8 78.5 mm to (126.2, 97.7), turned to -90 degrees
- moved H3 77.2 mm to (122.2, 147.3)
- moved IC4 75.8 mm to (155.7, 94.1)
- moved IC3 70.7 mm to (156.3, 100.9), turned to 180 degrees
- moved R55 70.1 mm to (160.8, 104.7)
- moved X1 69.6 mm to (155.9, 106.1), turned to 180 degrees
- moved R54 68.4 mm to (149.2, 56.5)
- moved D2 67.7 mm to (129.6, 110.2)
- moved J16 62.8 mm to (131.9, 80.6), turned to 180 degrees
- moved H2 60.8 mm to (177.4, 54.5)
- moved J6 56.0 mm to (154.7, 114.9), turned to 180 degrees
- moved J18 55.5 mm to (126.2, 95.8), turned to 90 degrees
- moved J1 55.4 mm to (144.3, 120.6), turned to 180 degrees
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Connections:
- C77 pad 1: /OV_VOUT -> /OV_OUT
- R46 pad 2: /OV_VOUT -> /OV_OUT
- R50 pad 1: /STR -> /STR_TOP
- U1 pad 20: /VID_RX -> /STR_TOP
- U1 pad 21: /VID_TX -> /XSHUT5
- U1 pad 22: /VID_CH1 -> /XSHUT4
- U1 pad 23: /VID_CH2 -> /ICM_INT1
- U1 pad 25: /VID_CH3 -> /ICM_INT2
- U1 pad 54: /XSHUT2 -> /CAM_RX
- U1 pad 55: /XSHUT3 -> /CAM_TX
- U1 pad 57: /XSHUT4 -> /XSHUT2
- U1 pad 58: /XSHUT5 -> /XSHUT3
- U8 pad 10: /SPI_SCLK -> /SPI_SCK
Routing:
- net +5V: track 29.8 -> 233.0 mm, vias 16 -> 26
- net GND: track 78.9 -> 197.6 mm, vias 6 -> 74
- net /I2C_SDA: track 103.8 -> 221.4 mm, vias 5 -> 10
- net /SPI_TX: track 0.00 -> 112.7 mm, vias 0 -> 10
- net /I2C_SCL: track 102.7 -> 211.8 mm, vias 5 -> 7
- net /SPI_SCK: track 0.00 -> 106.3 mm, vias 0 -> 8
- net /SPI_RX: track 0.00 -> 103.4 mm, vias 0 -> 8
- net +3V3: track 58.7 -> 155.2 mm, vias 35 -> 58
- net /I_SENSE: track 0.00 -> 54.6 mm, vias 0 -> 3
- net /VBAT: track 72.6 -> 126.8 mm, vias 8 -> 14
- net /GM_TX: track 0.00 -> 49.7 mm, vias 0 -> 2
- net /GM_PWM4: track 0.00 -> 49.3 mm, vias 0 -> 2
- net /GM_RX: track 0.00 -> 49.2 mm, vias 0 -> 2
- net /GM_PWM3: track 0.00 -> 44.3 mm, vias 0 -> 2
- net /GM_PWM1: track 0.00 -> 44.1 mm, vias 0 -> 2
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- added copper zone on F.Cu, net /OV_CLKIN
- added copper zone on B.Cu, net /VBAT
Other:
- board outline added: 60.4 x 98.2 mm
- board text added: "BOOT"
- board text added: "CHG RST"
- board text added: "RESET"
