File: dronePCB/dronePCB.kicad_pcb (KiCad board)
At the start: 6 copper layers, 60.4 x 98.2 mm, 205 parts, among them IC1 STUSB4500QTR, IC2 MP2338GTL-Z, IC3 BMI323, J1 BM03B-SRSS-TB, J10 DVR, J11 Strobe top, J12 Strobe bottom, J13 ToF400C, J14 ToF400C, J15 ToF400C, J16 ToF400C, J17 ToF400C, J18 DSHOT, J19 XT30, J2 USB_C_Receptacle, J20 MSD-1-A, J3 103AT-2 10k, J4 XT30, J5 JST, J6 Camera, J7 VID_ANT, J8 GEP-M10Q, J9 Avatar GMx, Q1 BSS138, Q2 BSS138, Q3 SQD40031EL_GE3, Q4 2N7002A, SW1 SW_BOOT, SW2 SW_RESET, SW3 SW_CHG_RST, SW4 CJS-1200TB1, SW5 CJS-1200TB1, SW6 CJS-1200TB1, SW7 SW_Push, U1 RP2350_80QFN, U11 LPS22HH, U2 W25Q128JVEIM TR, U3 APS6404L-3SQR-ZR, U4 BQ25792RQMR, U5 NCP1117-3.3_SOT223, U6 BQ76920PW, U7 E28-2G4M12SX, U8 AT7456E, U9 TX5823, Y1 ABM8-272-T3, Y2 ABM8W-27.0000MHZ-4-D1X-T3

Commit message: Finished the BoM
Parts:
- moved R11 0.30 mm to (140.3, 126.9)
- moved J20 0.10 mm to (130.4, 115.9)
Routing:
- net +3V3: track 155.6 -> 154.2 mm, vias 57 -> 56
- net GND: vias 527 -> 525
- net /SPI_SCK: vias 8 -> 7
- net /SPI_RX: vias 7 -> 6
Changed lines of the file:
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@@
 	(footprint "Resistor_SMD:R_0805_2012Metric_Pad1.20x1.40mm_HandSolder"
 		(layer "B.Cu")
-		(at 140.05 126.86 -90)
+		(at 140.35 126.91 -90)
 		(descr "Resistor SMD 0805 (2012 Metric), square (rectangular) end terminal, IPC-7351 nominal with elongated pad for handsoldering. (Body size source: IPC-SM-782 page 72, https://www.pcb-3d.com/wordpress/wp-content/uploads/ipc-sm-782a_amendment_1_and_2.pdf)")
 		(tags "resistor handsolder")
@@
 	(footprint "droneParts:MSD1A"
 		(layer "B.Cu")
-		(at 130.4 115.76 90)
+		(at 130.4 115.86 90)
 		(descr "MSD-1-A-1")
 		(tags "Connector")
@@
 	)
 	(via
-		(at 141.15 137.96)
-		(size 0.6)
-		(drill 0.3)
-		(layers "F.Cu" "B.Cu")
-		(free yes)
-		(capping no)
-		(covering
-			(front no)
-			(back no)
-		)
-		(plugging
-			(front no)
-			(back no)
-		)
-		(filling no)
-		(net "GND")
-	)
-	(via
 		(at 157.95 73.46)
 		(size 0.6)
@@
 	)
 	(via
-		(at 126.45 87.16)
-		(size 0.6)
-		(drill 0.3)
-		(layers "F.Cu" "B.Cu")
-		(free yes)
-		(net "GND")
-	)
-	(via
 		(at 179.35 71.21)
 		(size 0.6)
@@
 	)
 	(segment
-		(start 157.3 94.91)
-		(end 158.9 96.51)
-		(width 0.2)
-		(layer "F.Cu")
-		(net "+3V3")
-	)
-	(segment
 		(start 128.8875 72.45)
 		(end 128.8875 71.8925)
@@
 	)
 	(segment
-		(start 156.6 94.91)
-		(end 157.3 94.91)
-		(width 0.2)
-		(layer "F.Cu")
-		(net "+3V3")
-	)
-	(segment
 		(start 132.4 81.8175)
 		(end 132.84625 82.26375)
@@
 	)
 	(segment
-		(start 159.2 90.05)
-		(end 160.5275 90.05)
-		(width 0.2)
-		(layer "F.Cu")
-		(net "+3V3")
-	)
-	(segment
 		(start 142.8875 100.76)
 		(end 142.6875 100.56)
@@
 	)
 	(segment
-		(start 160.5275 90.05)
-		(end 160.55 90.0725)
+		(start 158.5 96.51)
+		(end 158.9 96.51)
+		(width 0.2)
+		(layer "F.Cu")
+		(net "+3V3")
+	)
+	(segment
+		(start 156.9 94.91)
+		(end 158.5 96.51)
 		(width 0.2)
 		(layer "F.Cu")
@@
 	)
 	(segment
+		(start 156.6 94.91)
+		(end 156.9 94.91)
+		(width 0.2)
+		(layer "F.Cu")
+		(net "+3V3")
+	)
+	(segment
 		(start 139.6875 92.96)
 		(end 140.0875 93.36)
@@
 	)
 	(via
-		(at 159.2 90.05)
-		(size 0.6)
-		(drill 0.3)
-		(layers "F.Cu" "B.Cu")
-		(capping no)
-		(covering
-			(front no)
-			(back no)
-		)
-		(plugging
-			(front no)
-			(back no)
-		)
-		(filling no)
-		(net "+3V3")
-	)
-	(via
 		(at 134.8375 98.84429)
 		(size 0.6)
@@
 	)
 	(segment
-		(start 155.7 105.56)
-		(end 158.1625 105.56)
-		(width 0.2)
-		(layer "F.Cu")
-		(net "/OV_CLKIN")
-	)
-	(segment
-		(start 158.1625 105.56)
-		(end 158.5 105.2225)
-		(width 0.2)
-		(layer "F.Cu")
-		(net "/OV_CLKIN")
-	)
-	(segment
 		(start 157 76.3225)
 		(end 155.5 76.3225)
@@
 	)
 	(via
-		(at 151 99.19)
-		(size 0.6)
-		(drill 0.3)
-		(layers "F.Cu" "B.Cu")
-		(capping no)
-		(covering
-			(front no)
-			(back no)
-		)
-		(plugging
-			(front no)
-			(back no)
-		)
-		(filling no)
-		(net "/SPI_RX")
-	)
-	(via
 		(at 151.77 108.99)
 		(size 0.6)
@@
 	)
 	(via
-		(at 149.951807 98.23)
-		(size 0.6)
-		(drill 0.3)
-		(layers "F.Cu" "B.Cu")
-		(capping no)
-		(covering
-			(front no)
-			(back no)
-		)
-		(plugging
-			(front no)
-			(back no)
-		)
-		(filling no)
-		(net "/SPI_SCK")
-	)
-	(via
 		(at 136.11 117.91)
 		(size 0.6)
@@
 	)
 	(segment
+		(start 150.7865 107.161)
+		(end 150.6 107.3475)
+		(width 0.2)
+		(layer "F.Cu")
+		(net "/OV_XFB")
+	)
+	(segment
+		(start 153.5 107.161)
+		(end 150.7865 107.161)
+		(width 0.2)
+		(layer "F.Cu")
+		(net "/OV_XFB")
+	)
+	(segment
 		(start 150.375 83.36)
 		(end 150.375 84.005)
@@
 	)
 	(segment
+		(start 155.7 105.56)
+		(end 158.1625 105.56)
+		(width 0.2)
+		(layer "F.Cu")
+		(net "/OV_CLKIN")
+	)
+	(segment
+		(start 158.1625 105.56)
+		(end 158.5 105.2225)
+		(width 0.2)
+		(layer "F.Cu")
+		(net "/OV_CLKIN")
+	)
+	(segment
 		(start 166.9 92.86)
 		(end 167.05 92.86)
@@
 	)
 	(segment
-		(start 139.64262 121.22988)
-		(end 139.6725 121.2)
-		(width 0.5)
-		(layer "B.Cu")
-		(net "Net-(J20-DAT1)")
-	)
-	(segment
-		(start 137.53219 121.22988)
-		(end 139.64262 121.22988)
-		(width 0.5)
-		(layer "B.Cu")
-		(net "Net-(J20-DAT1)")
-	)
-	(segment
 		(start 137.53219 113.529982)
 		(end 137.932172 113.13)
@@
 	)
 	(segment
-		(start 150.7865 107.161)
-		(end 150.6 107.3475)
-		(width 0.2)
-		(layer "F.Cu")
-		(net "/OV_XFB")
+		(start 139.64262 121.22988)
+		(end 139.6725 121.2)
+		(width 0.5)
+		(layer "B.Cu")
+		(net "Net-(J20-DAT1)")
 	)
 	(segment
-		(start 153.5 107.161)
-		(end 150.7865 107.161)
-		(width 0.2)
-		(layer "F.Cu")
-		(net "/OV_XFB")
+		(start 137.53219 121.22988)
+		(end 139.64262 121.22988)
+		(width 0.5)
+		(layer "B.Cu")
+		(net "Net-(J20-DAT1)")
 	)
 	(zone
