File: dronePCB/dronePCB.kicad_sch (KiCad schematic)
At the start: 73 parts, among them IC3 DPS368XTSA1, IC4 ICM-42688-P, J10 DVR, J11 Strobe top, J12 Strobe bottom, J13 ToF400C, J14 ToF400C, J15 ToF400C, J16 ToF400C, J17 ToF400C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

Commit message: Started filling the BoM and changed some components
Parts:
- removed IC3: DPS368XTSA1, droneParts:DPS368XTSA1, symbol DPS368XTSA1:DPS368XTSA1
- removed IC4: ICM-42688-P, droneParts:IIM42352, symbol ICM-42688-P:ICM-42688-P
- removed R35: 10k, Resistor_SMD:R_0805_2012Metric_Pad1.20x1.40mm_HandSolder, symbol Device:R
- added IC3: BMI323, droneParts:BMI323, symbol BMI323:BMI323
- added U11: LPS22HH, Package_LGA:ST_HLGA-10_2x2mm_P0.5mm_LayoutBorder3x2y, symbol Sensor_Pressure:LPS22HH
- C66, C67, C68, C69, C70, C71, C72, C73, C74, C77, C79, C81, C83, C84, C85, C86, C87, C88: Link (none) -> https://www.mouser.pl/ProductDetail/KYOCERA-AVX/08056D104KA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; Manufacturer_Part_Number (none) -> 08056D104KAT2A; Price per unit (none) -> 0.031
- C75, C76: Link (none) -> https://www.mouser.pl/ProductDetail/Walsin/0805N220J500CT?q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; Manufacturer_Part_Number (none) -> 0805N220J500CT; Price per unit (none) -> 0.126
- C78: footprint Capacitor_SMD:C_Elec_3x5.4 -> droneParts:CAPAE830X1080N; Link (none) -> https://www.mouser.pl/ProductDetail/Nichicon/UCW1C471MNL1GS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; Manufacturer_Part_Number (none) -> UCW1C471MNL1GS; Price per unit (none) -> 0.62
- C80, C82: Link (none) -> https://www.mouser.pl/ProductDetail/Samsung-Electro-Mechani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; Manufacturer_Part_Number (none) -> CL21B105KAFNNNG; Price per unit (none) -> 0.034
- C89: value 0.1uf -> 100n; Link (none) -> https://www.mouser.pl/ProductDetail/KYOCERA-AVX/08056D104KA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; Manufacturer_Part_Number (none) -> 08056D104KAT2A; Price per unit (none) -> 0.031
- C90: value 10uF -> 10u; Link (none) -> https://www.mouser.pl/ProductDetail/Samsung-Electro-Mechani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; Manufacturer_Part_Number (none) -> CL21A106KOQNNNE; Price per unit (none) -> 0.015
- D2, D3: Link (none) -> https://www.mouser.pl/ProductDetail/onsemi/MBR0530T1G?qs=3J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; Manufacturer_Part_Number (none) -> MBR0530T1G; Price per unit (none) -> 0.45
- D4: value LED -> BLUE; Link (none) -> https://www.mouser.pl/ProductDetail/Wurth-Elektronik/150080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; Manufacturer_Part_Number (none) -> 150080BS75000; Price per unit (none) -> 0.19
- H1, H2, H3, H4: Link (none) -> n/a; Manufacturer_Part_Number (none) -> n/a; Price per unit (none) -> n/a
Connections:
- net +3V3: now also IC3.12 (CSB), IC3.5 (VDDIO), IC3.8 (VDD), U11.1 (Vdd_IO), U11.10 (VDD)
- net DPS_CS: now also U11.6 (~{CS})
- net GND: now also IC3.1 (SDO), IC3.6 (GNDIO), IC3.7 (GND), U11.3 (GND), U11.8 (GND), U11.9 (GND)
- net I2C_SCL: now also IC3.14 (SDX)
- net I2C_SDA: now also IC3.13 (SCX)
- net SPI_RX: now also U11.5 (SA0)
- net SPI_SCK: now also U11.2 (SCL)
- net SPI_TX: now also U11.4 (SDA)
- new net BMI_INT1: IC3.4 (INT1)
- new net BMI_INT2: IC3.9 (INT2)
- new net LPSINT: U11.7 (INT_DRDY)
- no-connect marks 17 -> 20
Other:
- note removed: "IMU"
- moved on the sheet: C84, J13

Commit message: Added more information to BoM
Parts:
- removed R55: 10k, Resistor_SMD:R_0805_2012Metric_Pad1.20x1.40mm_HandSolder, symbol Device:R
- removed U10: TF-01A, droneParts:TF-01A, symbol TF-01A:TF-01A
- removed X1: OT2EL4C4JI-111OLP-27M, droneParts:OT2EL4C4JI-111OLP-27M, symbol OT2EL4C4JI-111OLP-27M:OT2EL4C4JI-111OLP-27M
- added J20: MSD-1-A, droneParts:MSD1A, symbol MSD-1-A:MSD-1-A
- added Y2: ABM8W-27.0000MHZ-4-D1X-T3, droneParts:ABM8W480000MHZ6D1XT3, symbol Device:Crystal_GND24
- C89: value 100n -> 2p; Link https://www.mouser.pl/ProductDetail/KYOCERA-AVX/08056D104KA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 -> https://www.mouser.pl/ProductDetail/Walsin/0805N2R0C500CT?q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; Manufacturer_Part_Number 08056D104KAT2A -> 0805N2R0C500CT; Price per unit 0.031 -> 0.151
- C90: value 10u -> 2p; Link https://www.mouser.pl/ProductDetail/Samsung-Electro-Mechani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 -> https://www.mouser.pl/ProductDetail/Walsin/0805N2R0C500CT?q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; Manufacturer_Part_Number CL21A106KOQNNNE -> 0805N2R0C500CT; Price per unit 0.015 -> 0.151
- H1, H2, H3, H4: Price per unit n/a -> 0
- J10: Link (none) -> https://www.mouser.pl/ProductDetail/JST-Commercial/B3B-PH-S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; Manufacturer_Part_Number (none) -> B3B-PH-SM4-TB(LF)(SN); Price per unit (none) -> 0.52
- J11, J12: Link (none) -> https://www.mouser.pl/ProductDetail/JST-Commercial/B2B-PH-S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; Manufacturer_Part_Number (none) -> B2B-PH-SM4-TB(LF)(SN); Price per unit (none) -> 0.47
- J13, J14, J15, J16, J17, J8: Link (none) -> https://www.mouser.pl/ProductDetail/JST-Commercial/B6B-PH-S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; Manufacturer_Part_Number (none) -> B6B-PH-SM4-TB(LF)(SN); Price per unit (none) -> 0.761
- J18, J9: Link (none) -> https://www.mouser.pl/ProductDetail/JST-Commercial/B8B-PH-S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; Manufacturer_Part_Number (none) -> B8B-PH-SM4-TBT(LF)(SN); Price per unit (none) -> 1.01
- J19: Link (none) -> https://www.tme.eu/pl/details/xt30u-f/zlacza-dc/amass/; Manufacturer_Part_Number (none) -> XT30U-F AMASS; Price per unit (none) -> 0.45
- J6: Link (none) -> https://www.mouser.pl/ProductDetail/JST-Commercial/B5B-PH-S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; Manufacturer_Part_Number (none) -> B5B-PH-SM4-TB(LF)(SN); Price per unit (none) -> 0.70
- J7: Link (none) -> n/a; Manufacturer_Part_Number (none) -> n/a; Price per unit (none) -> 0
- Q1, Q2: Link (none) -> https://www.mouser.pl/ProductDetail/onsemi/BSS138?qs=HK%252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; Manufacturer_Part_Number (none) -> BSS138; Price per unit (none) -> 0.361
- SW4, SW5, SW6: Link (none) -> https://www.mouser.pl/ProductDetail/Nidec-Components/CJS-12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; Price per unit (none) -> 0.89
- U7: Link (none) -> https://pl.aliexpress.com/item/1005007803684660.html?spm=a2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; Manufacturer_Part_Number (none) -> E28-2G4M12SX; Price per unit (none) -> 7.11
- U8: Link (none) -> https://pl.aliexpress.com/item/1005009996756170.html?spm=a2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; Manufacturer_Part_Number (none) -> AT7456E; Price per unit (none) -> 3.15
- U9: Link (none) -> https://pl.aliexpress.com/item/1005011789861750.html?spm=a2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; Manufacturer_Part_Number (none) -> TX5823; Price per unit (none) -> 17.18
Connections:
- net +3V3: now also R48.2, J20.4 (VDD); no longer C89.1, C90.1, R48.1
- net GND: now also C89.1, J20.10 (GND_2), J20.11 (GND_3), J20.12 (GND_4), J20.6 (VSS), J20.9 (GND_1), Y2.2 (G), Y2.4 (G); no longer C89.2
- net OV_CLKIN: now also C90.1, Y2.1
- net SD_CD: now also J20.CD1
- net SD_CS: now also J20.2 (CD/DAT3)
- net SPI_RX: now also J20.7 (DAT0)
- net SPI_SCK: now also J20.5 (CLK)
- net SPI_TX: now also J20.3 (CMD)
- net OV_XFB: now reaches U8.6 (XFB)
- net OV_XFB: now also C89.2, Y2.3
- net at R47.2: now also J20.1 (DAT2)
- new net: J20.8 (DAT1), R48.1
- no-connect marks 20 -> 19

Commit message: Finished the BoM
Parts:
- R42, R43, R44, R50, R52: Link (none) -> https://www.mouser.pl/ProductDetail/Bourns/CRM0805-FX-1001E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; Manufacturer_Part_Number (none) -> CRM0805-FX-1001ELF; Price per unit (none) -> 0.10
- R45, R46: Link (none) -> https://www.mouser.pl/ProductDetail/Vishay/CRCW080575R0FKEA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; Manufacturer_Part_Number (none) -> CRCW080575R0FKEA; Price per unit (none) -> 0.10
- R47, R48, R49: Link (none) -> https://www.mouser.pl/ProductDetail/Susumu/RG2012P-472-B-T5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; Manufacturer_Part_Number (none) -> RG2012P-472-B-T5; Price per unit (none) -> 0.10
- R51, R53: Link (none) -> https://www.mouser.pl/ProductDetail/Bourns/CRM0805-FX-1002E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; Manufacturer_Part_Number (none) -> CRM0805-FX-1002ELF; Price per unit (none) -> 0.041
- R54: Link (none) -> https://www.mouser.pl/ProductDetail/Vishay/CRCW0805220RFKEA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; Manufacturer_Part_Number (none) -> CRCW0805220RFKEA; Price per unit (none) -> 0.10
