File: dronePCB/powerCircuit.kicad_sch (KiCad schematic)
At the start: 91 parts, among them IC1 STUSB4500QTR, IC2 MP2338GTL-Z, J3 103AT-2 10k, J4 XT30, J5 JST, Q3 SQD40031EL_GE3, Q4 2N7002A, SW3 SW_CHG_RST, SW7 SW_Push, U4 BQ25792RQMR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

Commit message: Started filling the BoM and changed some components
Parts:
- C22, C23, C24, C27, C54, C55, C56, C57, C59, C60, C61: Link (none) -> https://www.mouser.pl/ProductDetail/Samsung-Electro-Mechani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; Manufacturer_Part_Number (none) -> CL21B105KAFNNNG; Price per unit (none) -> 0.034
- C25, C30, C31, C32, C34, C35, C36, C37, C38, C40, C41, C52, C53: Link (none) -> https://www.mouser.pl/ProductDetail/Samsung-Electro-Mechani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; Manufacturer_Part_Number (none) -> CL21A106KOQNNNE; Price per unit (none) -> 0.015
- C26, C33, C39, C46, C47, C62, C63, C64: Link (none) -> https://www.mouser.pl/ProductDetail/KYOCERA-AVX/08056D104KA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; Manufacturer_Part_Number (none) -> 08056D104KAT2A; Price per unit (none) -> 0.031
- C28, C29: Link (none) -> https://www.mouser.pl/ProductDetail/KYOCERA-AVX/KGM21NR71C4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; Manufacturer_Part_Number (none) -> KGM21NR71C473KT; Price per unit (none) -> 0.10
- C42: Link (none) -> https://www.mouser.pl/ProductDetail/Samsung-Electro-Mechani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; Manufacturer_Part_Number (none) -> CL21B102KBCNNNC; Price per unit (none) -> 0.10
- C44, C48, C49: Link (none) -> https://www.mouser.pl/ProductDetail/Samsung-Electro-Mechani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; Manufacturer_Part_Number (none) -> CL21A226KQCLRNC; Price per unit (none) -> 0.14
- C45: footprint Capacitor_SMD:C_Elec_3x5.4 -> droneParts:CAPAE830X1080N; Link (none) -> https://www.mouser.pl/ProductDetail/Nichicon/UCW1C471MNL1GS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; Manufacturer_Part_Number (none) -> UCW1C471MNL1GS; Price per unit (none) -> 0.62
- C50: Link (none) -> https://www.mouser.pl/ProductDetail/Walsin/0805N301J500CT?q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; Manufacturer_Part_Number (none) -> 0805N301J500CT; Price per unit (none) -> 0.138
- C51: Link (none) -> https://www.mouser.pl/ProductDetail/YAGEO/CC0805KRX7R7BB223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; Manufacturer_Part_Number (none) -> CC0805KRX7R7BB223; Price per unit (none) -> 0.10
- D5: Link (none) -> https://www.mouser.pl/ProductDetail/onsemi/MMSZ4699T1G?qs=P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; Manufacturer_Part_Number (none) -> MMSZ4699T1G; Price per unit (none) -> 0.10
- IC1: Link (none) -> https://www.mouser.pl/ProductDetail/STMicroelectronics/STUS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; Price per unit (none) -> 1.97
- IC2: Link (none) -> https://www.mouser.pl/ProductDetail/Monolithic-Power-System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; Price per unit (none) -> 1.55

Commit message: Added more information to BoM
Parts:
- J3: Link (none) -> https://www.mouser.pl/ProductDetail/JST-Commercial/B2B-PH-S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; Manufacturer_Part_Number (none) -> B2B-PH-SM4-TB(LF)(SN); Price per unit (none) -> 0.47
- J4: Link (none) -> https://www.tme.eu/pl/details/xt30u-f/zlacza-dc/amass/; Manufacturer_Part_Number (none) -> XT30U-F AMASS; Price per unit (none) -> 0.45
- J5: Link (none) -> https://www.mouser.pl/ProductDetail/JST-Commercial/B5B-PH-S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; Manufacturer_Part_Number (none) -> B5B-PH-SM4-TB(LF)(SN); Price per unit (none) -> 0.70
- L2: Link (none) -> https://www.mouser.pl/ProductDetail/ABRACON/AMPLH7020S-1R0M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; Manufacturer_Part_Number (none) -> AMPLH7020S-1R0MT; Price per unit (none) -> 0.82
- L3: Link (none) -> https://www.mouser.pl/ProductDetail/ABRACON/AMPLH5030S-6R8M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; Manufacturer_Part_Number (none) -> AMPLH5030S-6R8MT; Price per unit (none) -> 0.92
- Q3: Link (none) -> https://www.mouser.pl/ProductDetail/Vishay-Semiconductors/S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; Price per unit (none) -> 2.34
- SW3: Link (none) -> https://www.mouser.pl/ProductDetail/Wurth-Elektronik/434133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; Manufacturer_Part_Number (none) -> 434133025816; Price per unit (none) -> 0.55
- SW7: Link (none) -> https://www.mouser.pl/ProductDetail/Alps-Alpine/SKRTLAE010?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; Manufacturer_Part_Number (none) -> SKRTLAE010; Price per unit (none) -> 0.427
- U4: Link (none) -> https://www.mouser.pl/ProductDetail/Texas-Instruments/BQ257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; Manufacturer_Part_Number (none) -> BQ25792RQMR; Price per unit None -> 6.84
- U5: Link (none) -> https://www.mouser.pl/ProductDetail/onsemi/NCP1117ST33T3G?q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; Manufacturer_Part_Number (none) -> NCP1117ST33T3G; Price per unit (none) -> 0.58
- U6: Link (none) -> https://www.mouser.pl/ProductDetail/Texas-Instruments/BQ769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; Manufacturer_Part_Number (none) -> BQ7692000PW; Price per unit (none) -> 4.19

Commit message: Finished the BoM
Parts:
- Q4: Link (none) -> https://www.mouser.pl/ProductDetail/Diotec-Semiconductor/2N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; Manufacturer_Part_Number (none) -> 2N7002A; Price per unit (none) -> 0.14
- R13, R14, R15, R16, R17, R19, R26, R28, R40, R59: Link (none) -> https://www.mouser.pl/ProductDetail/Bourns/CRM0805-FX-1002E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; Manufacturer_Part_Number (none) -> CRM0805-FX-1002ELF; Price per unit (none) -> 0.041
- R18, R37, R38, R41: Link (none) -> https://www.mouser.pl/ProductDetail/SEI-Stackpole/RMCA0805F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; Manufacturer_Part_Number (none) -> RMCA0805FT100R-HP; Price per unit (none) -> 0.10
- R20: Link (none) -> https://www.mouser.pl/ProductDetail/YAGEO/RT0805FRE075K23L?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; Manufacturer_Part_Number (none) -> RT0805FRE075K23L; Price per unit (none) -> 0.10
- R21: Link (none) -> n/a; Manufacturer_Part_Number (none) -> n/a; Price per unit (none) -> 0
- R22: Link (none) -> https://www.mouser.pl/ProductDetail/YAGEO/RT0805DRE0730K1L?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; Manufacturer_Part_Number (none) -> RT0805DRE0730K1L; Price per unit (none) -> 0.10
- R23: Link (none) -> https://www.mouser.pl/ProductDetail/Bourns/CR0805-FX-1742EL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; Manufacturer_Part_Number (none) -> CR0805-FX-1742ELF; Price per unit (none) -> 0.10
- R24: Link (none) -> https://www.mouser.pl/ProductDetail/YAGEO/RT0805FRE07127KL?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; Manufacturer_Part_Number (none) -> RT0805FRE07127KL; Price per unit (none) -> 0.11
- R25, R56: Link (none) -> https://www.mouser.pl/ProductDetail/Bourns/CR0805AFX-1003EA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; Manufacturer_Part_Number (none) -> CR0805AFX-1003EAS; Price per unit (none) -> 0.10
- R27: Link (none) -> https://www.mouser.pl/ProductDetail/YAGEO/RT0805FRE0790K9L?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; Manufacturer_Part_Number (none) -> RT0805FRE0790K9L; Price per unit (none) -> 0.10
- R29: Link (none) -> https://www.mouser.pl/ProductDetail/YAGEO/RT0805FRE07191KL?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; Manufacturer_Part_Number (none) -> RT0805FRE07191KL; Price per unit (none) -> 0.10
- R30: Link (none) -> https://www.mouser.pl/ProductDetail/YAGEO/RT0805FRD0749K9L?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; Manufacturer_Part_Number (none) -> RT0805FRD0749K9L; Price per unit (none) -> 0.10
- R31, R32, R33, R34, R36, R57, R58: Link (none) -> https://www.mouser.pl/ProductDetail/Bourns/CRM0805-FX-1001E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; Manufacturer_Part_Number (none) -> CRM0805-FX-1001ELF; Price per unit (none) -> 0.10
- R39: Link (none) -> https://www.mouser.pl/ProductDetail/SEI-Stackpole/CSSH0805F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; Manufacturer_Part_Number (none) -> CSSH0805FT1L00; Price per unit (none) -> 0.60
