File: dronePCB/backup/untitled.kicad_sch (KiCad schematic)
At the start: 43 parts, among them J1 BM03B-SRSS-TB, J2 USB_C_Receptacle, SW1 SW_BOOT, SW2 SW_RESET, U1 RP2350_80QFN, U2 W25Q128JVPIQ, U3 APS6404L-3SQR-ZR, Y1 ABM8-272-T3

Commit message: Added power switch
Parts:
- C1, C16: footprint Capacitor_SMD:C_0805_2012Metric_Pad1.18x1.45mm_HandSolder -> (none); Link https://www.mouser.pl/ProductDetail/Samsung-Electro-Mechani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 -> (none); Manufacturer_Part_Number CL21A475KPFNNNF -> (none); Price per unit 0.10 -> (none)
- C10, C11, C12, C13, C14, C15, C17, C18, C19, C20, C21, C4, C5, C6, C7, C8, C9: footprint Capacitor_SMD:C_0805_2012Metric_Pad1.18x1.45mm_HandSolder -> (none)
- C2, C3: footprint Capacitor_SMD:C_0402_1005Metric_Pad0.74x0.62mm_HandSolder -> (none); Link https://www.mouser.pl/ProductDetail/Samsung-Electro-Mechani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 -> (none); Manufacturer_Part_Number CL05A475KQ5NRNC -> (none); Price per unit 0.12 -> (none)
- D1: footprint Diode_SMD:D_SOD-323_HandSoldering -> (none)
- J1: footprint Connector_JST:JST_SH_BM03B-SRSS-TB_1x03-1MP_P1.00mm_Vertical -> (none)
- J2: footprint Connector_USB:USB_C_Receptacle_Amphenol_12401610E4-2A -> (none)
- L1: footprint droneParts:AOTAB201610S3R3101T -> (none)
- R1, R10, R11, R12, R2, R3, R4, R5, R6, R7, R8, R9: footprint Resistor_SMD:R_0805_2012Metric_Pad1.20x1.40mm_HandSolder -> (none)
- SW1, SW2: footprint Button_Switch_SMD:SW_Push_1P1T_NO_Vertical_Wuerth_434133025816 -> (none)
- U1: footprint MCU:RP2350B -> RP2350_80QFN_minimal:RP2350-QFN-80-1EP_10x10_P0.4mm_EP3.4x3.4mm_ThermalVias
- U2: footprint Flash:W25Q128JVPIQ -> W25Q128JVPIQ:W25Q128JVPIQ; Price (none) -> None; Price per unit None -> (none)
- U3: footprint droneParts:PSON50P200X300X50-9N -> APS6404L-3SQR-ZR:PSON50P200X300X50-9N; Price (none) -> None; Price per unit None -> (none)
- Y1: footprint droneParts:ABM8272T3 -> (none)
Connections:
- net GPIO4 renamed USB_MODE3
- net GPIO5 renamed USB_MODE2
Other:
- sheet Power Circuit ports: added USB_MODE2, USB_MODE3; removed PWR
- company: Author: Mejpek -> (none)
- title: RP2350B -> (none)
